Commit message: first commit

File: robots/hand.xacro (robot description, xacro)
@@ -22,5 +22,5 @@
         </geometry>
       </collision>
-      <collision>
+      <!--<collision>
         <origin xyz="0 -0.05 0.04" rpy="0 0 0"/>
         <geometry>
@@ -51,5 +51,5 @@
           <sphere radius="${0.02+safety_distance}"/>
         </geometry>
-      </collision>
+      </collision> -->
       <inertial>
         <origin xyz="0 0 0" rpy="0 0 0" />
@@ -67,8 +67,15 @@
     <link name="${ns}_leftfinger">
       <visual>
+        <origin xyz="0 0 0" rpy="0 0 ${-pi}"/>
         <geometry>
           <mesh filename="$(find franka_description)/meshes/visual/finger.dae"/>
         </geometry>
       </visual>
+      <inertial>
+        <origin xyz="0 0 0" rpy="0 0 0" />
+        <mass value="0.02" />
+        <inertia ixx="0.000001667" ixy="0.0" ixz="0.0" iyy="0.000001667" iyz="0.0"
+            izz="0.000000667" />
+      </inertial>
     </link>
     <link name="${ns}_rightfinger">

File: robots/panda_arm.urdf.xacro (robot description, xacro)
@@ -8,11 +8,11 @@
   <link name="world" />
   <xacro:include filename="$(find franka_description)/robots/panda_arm.xacro"/>
-  <xacro:panda_arm arm_id="$(arg arm_id)" safety_distance="0.03"/>
+  <xacro:panda_arm arm_id="$(arg arm_id)" safety_distance="0.03" connected_to="world" />
   <xacro:if value="$(arg hand)">
     <xacro:include filename="$(find franka_description)/robots/hand.xacro"/>
     <xacro:hand ns="$(arg arm_id)" rpy="0 0 ${-pi/4}" connected_to="$(arg arm_id)_link8" safety_distance="0.03"/>
   </xacro:if>
-  <xacro:include filename="$(find franka_description)/robots/panda_arm.ros2_control.xacro"/>
-  <xacro:panda_arm_ros2_control ns="$(arg arm_id)" robot_ip="$(arg robot_ip)" use_fake_hardware="$(arg use_fake_hardware)" fake_sensor_commands="$(arg fake_sensor_commands)"/>
-  <xacro:include filename="$(find franka_description)/robots/panda.gazebo.xacro" />
+  <xacro:include filename="$(find franka_description)/robots/panda_arm_ros2_control.xacro"/>
+  <xacro:panda_arm_ros2_control ns="$(arg arm_id)" />
+  <xacro:include filename="$(find franka_description)/robots/panda_gazebo.xacro" />
 </robot>

File: robots/panda_arm.xacro (robot description, xacro)
@@ -32,5 +32,5 @@
     </inertial>
   </xacro:macro>
-  <xacro:macro name="panda_arm" params="arm_id:='panda' description_pkg:='franka_description' connected_to:='' xyz:='0 0 0' rpy:='0 0 0' safety_distance:=0">
+  <xacro:macro name="panda_arm" params="arm_id:='panda' description_pkg:='franka_description' connected_to:='' xyz:='0 0 0' rpy:='0 0 0' safety_distance:='' ">
     <xacro:unless value="${not connected_to}">
       <joint name="${arm_id}_joint_${connected_to}" type="fixed">
@@ -41,11 +41,11 @@
     </xacro:unless>
     <xacro:property
-    name="joint_damping" value="1.0" />
-    <joint name="robot_to_world" type="fixed">
+    name="joint_damping" value="10.0" />
+    <!--<joint name="robot_to_world" type="fixed">
       <parent link="world" />
       <child link="${arm_id}_link0" />
       <origin xyz="0.0 0.0 0.0" rpy="0.0 0.0 0.0" />
       <dynamics damping="${joint_damping}" />
-    </joint>
+    </joint>-->
     <link name="${arm_id}_link0">
       <visual>

File: robots/panda_arm_ros2_control.xacro (robot description, xacro)
@@ -6,5 +6,5 @@
     </plugin>
 </gazebo>
-  <xacro:macro name="panda_arm_ros2_control" params="ns robot_ip use_fake_hardware:=^|false fake_sensor_commands:=^|false">
+  <xacro:macro name="panda_arm_ros2_control" params="ns">
     <ros2_control name="GazeboSystem" type="system">
       <hardware>
@@ -17,5 +17,5 @@
           <state_interface name="position"/>
           <state_interface name="velocity"/>
-        <!--  <state_interface name="effort"/>  -->
+          <state_interface name="effort"/>
         </joint>
       </xacro:macro>

File: robots/panda_gazebo.xacro (robot description, xacro)
@@ -20,5 +20,5 @@
         <kp>0.0</kp>
         <kd>0.0</kd>
-        <min_depth>0</min_depth>
+        <min_depth>0.001</min_depth>
         <!-- <max_vel>0</max_vel> -->
         <slip1>0</slip1>
@@ -31,5 +31,5 @@
         <kp>0.0</kp>
         <kd>0.0</kd>
-        <min_depth>0</min_depth>
+        <min_depth>0.001</min_depth>
         <!-- <max_vel>0</max_vel> -->
         <slip1>0</slip1>
@@ -62,5 +62,5 @@
         <kp>100000.0</kp>
         <kd>100.0</kd>
-        <min_depth>0</min_depth>
+        <min_depth>0.001</min_depth>
         <!-- <max_vel>0</max_vel> -->
         <slip1>0.2</slip1>
@@ -73,5 +73,5 @@
         <kp>50000.0</kp>
         <kd>1.0</kd>
-        <min_depth>0</min_depth>
+        <min_depth>0.001</min_depth>
         <!-- <max_vel>0</max_vel> -->
         <slip1>0</slip1>
